Commit message: add gazebo and moveit_config for tm1100, tm1300

File: tm_description/urdf/tm1100.urdf.xacro (robot description, xacro)
@@ -57,5 +57,5 @@
       <visual>
         <geometry>
-	  <mesh filename="package://tm_description/meshes/tm1100/visual/Base.STL" />
+	  <mesh filename="package://tm_description/meshes/tm1100/visual/Base.dae" />
         </geometry>
         <material name="Grey">
@@ -75,5 +75,5 @@
       <visual>
         <geometry>
-	  <mesh filename="package://tm_description/meshes/tm1100/visual/Shoulder1.STL" />
+	  <mesh filename="package://tm_description/meshes/tm1100/visual/Shoulder1.dae" />
         </geometry>
         <material name="DarkOlive">
@@ -106,5 +106,5 @@
       <visual>
         <geometry>
-	  <mesh filename="package://tm_description/meshes/tm1100/visual/Arm1.STL" />
+	  <mesh filename="package://tm_description/meshes/tm1100/visual/Arm1.dae" />
         </geometry>
         <material name="DarkOlive">
@@ -137,5 +137,5 @@
       <visual>
         <geometry>
-	  <mesh filename="package://tm_description/meshes/tm1100/visual/Arm2.STL" />
+	  <mesh filename="package://tm_description/meshes/tm1100/visual/Arm2.dae" />
         </geometry>
         <material name="DarkOlive">
@@ -168,5 +168,5 @@
       <visual>
         <geometry>
-	  <mesh filename="package://tm_description/meshes/tm1100/visual/Wrist1.STL" />
+	  <mesh filename="package://tm_description/meshes/tm1100/visual/Wrist1.dae" />
         </geometry>
         <material name="DarkOlive">
@@ -199,5 +199,5 @@
       <visual>
         <geometry>
-	  <mesh filename="package://tm_description/meshes/tm1100/visual/Wrist2.STL" />
+	  <mesh filename="package://tm_description/meshes/tm1100/visual/Wrist2.dae" />
         </geometry>
         <material name="DarkOlive">
@@ -230,5 +230,5 @@
       <visual>
         <geometry>
-	  <mesh filename="package://tm_description/meshes/tm1100/visual/Wrist3.STL" />
+	  <mesh filename="package://tm_description/meshes/tm1100/visual/Wrist3.dae" />
         </geometry>
 	<origin xyz="0 0 0.015" rpy="0 0 0"/>

File: tm_description/urdf/tm1300.urdf.xacro (robot description, xacro)
@@ -56,5 +56,5 @@
       <visual>
         <geometry>
-	  <mesh filename="package://tm_description/meshes/tm1300/visual/Base.STL" />
+	  <mesh filename="package://tm_description/meshes/tm1300/visual/Base.dae" />
         </geometry>
         <material name="Grey">
@@ -74,5 +74,5 @@
       <visual>
         <geometry>
-	  <mesh filename="package://tm_description/meshes/tm1300/visual/Shoulder1.STL" />
+	  <mesh filename="package://tm_description/meshes/tm1300/visual/Shoulder1.dae" />
         </geometry>
         <material name="DarkOlive">
@@ -105,5 +105,5 @@
       <visual>
         <geometry>
-	  <mesh filename="package://tm_description/meshes/tm1300/visual/Arm1.STL" />
+	  <mesh filename="package://tm_description/meshes/tm1300/visual/Arm1.dae" />
         </geometry>
         <material name="DarkOlive">
@@ -136,5 +136,5 @@
       <visual>
         <geometry>
-	  <mesh filename="package://tm_description/meshes/tm1300/visual/Arm2.STL" />
+	  <mesh filename="package://tm_description/meshes/tm1300/visual/Arm2.dae" />
         </geometry>
         <material name="DarkOlive">
@@ -167,5 +167,5 @@
       <visual>
         <geometry>
-	  <mesh filename="package://tm_description/meshes/tm1300/visual/Wrist1.STL" />
+	  <mesh filename="package://tm_description/meshes/tm1300/visual/Wrist1.dae" />
         </geometry>
         <material name="DarkOlive">
@@ -198,5 +198,5 @@
       <visual>
         <geometry>
-	  <mesh filename="package://tm_description/meshes/tm1300/visual/Wrist2.STL" />
+	  <mesh filename="package://tm_description/meshes/tm1300/visual/Wrist2.dae" />
         </geometry>
         <material name="DarkOlive">
@@ -229,5 +229,5 @@
       <visual>
         <geometry>
-	  <mesh filename="package://tm_description/meshes/tm1300/visual/Wrist3.STL" />
+	  <mesh filename="package://tm_description/meshes/tm1300/visual/Wrist3.dae" />
         </geometry>
 	<origin xyz="0 0 0.015" rpy="0 0 0"/>

File: tm_description/urdf/tm700.urdf.xacro (robot description, xacro)
@@ -57,5 +57,5 @@
       <visual>
         <geometry>
-	  <mesh filename="package://tm_description/meshes/tm700/visual/Base.STL" />
+	  <mesh filename="package://tm_description/meshes/tm700/visual/Base.dae" />
         </geometry>
         <material name="Grey">
@@ -75,5 +75,5 @@
       <visual>
         <geometry>
-	  <mesh filename="package://tm_description/meshes/tm700/visual/Shoulder1.STL" />
+	  <mesh filename="package://tm_description/meshes/tm700/visual/Shoulder1.dae" />
         </geometry>
         <material name="DarkOlive">
@@ -106,5 +106,5 @@
       <visual>
         <geometry>
-	  <mesh filename="package://tm_description/meshes/tm700/visual/Arm1.STL" />
+	  <mesh filename="package://tm_description/meshes/tm700/visual/Arm1.dae" />
         </geometry>
         <material name="DarkOlive">
@@ -137,5 +137,5 @@
       <visual>
         <geometry>
-	  <mesh filename="package://tm_description/meshes/tm700/visual/Arm2.STL" />
+	  <mesh filename="package://tm_description/meshes/tm700/visual/Arm2.dae" />
         </geometry>
         <material name="DarkOlive">
@@ -168,5 +168,5 @@
       <visual>
         <geometry>
-	  <mesh filename="package://tm_description/meshes/tm700/visual/Wrist1.STL" />
+	  <mesh filename="package://tm_description/meshes/tm700/visual/Wrist1.dae" />
         </geometry>
         <material name="DarkOlive">
@@ -199,5 +199,5 @@
       <visual>
         <geometry>
-	  <mesh filename="package://tm_description/meshes/tm700/visual/Wrist2.STL" />
+	  <mesh filename="package://tm_description/meshes/tm700/visual/Wrist2.dae" />
         </geometry>
         <material name="DarkOlive">
@@ -230,5 +230,5 @@
       <visual>
         <geometry>
-	  <mesh filename="package://tm_description/meshes/tm700/visual/Wrist3.STL" />
+	  <mesh filename="package://tm_description/meshes/tm700/visual/Wrist3.dae" />
         </geometry>
 	<origin xyz="0 0 0.015" rpy="0 0 0"/>

File: tm_description/urdf/tm900.urdf.xacro (robot description, xacro)
@@ -56,5 +56,5 @@
       <visual>
         <geometry>
-	  <mesh filename="package://tm_description/meshes/tm900/visual/Base.STL" />
+	  <mesh filename="package://tm_description/meshes/tm900/visual/Base.dae" />
         </geometry>
         <material name="Grey">
@@ -74,5 +74,5 @@
       <visual>
         <geometry>
-	  <mesh filename="package://tm_description/meshes/tm900/visual/Shoulder1.STL" />
+	  <mesh filename="package://tm_description/meshes/tm900/visual/Shoulder1.dae" />
         </geometry>
         <material name="DarkOlive">
@@ -105,5 +105,5 @@
       <visual>
         <geometry>
-	  <mesh filename="package://tm_description/meshes/tm900/visual/Arm1.STL" />
+	  <mesh filename="package://tm_description/meshes/tm900/visual/Arm1.dae" />
         </geometry>
         <material name="DarkOlive">
@@ -136,5 +136,5 @@
       <visual>
         <geometry>
-	  <mesh filename="package://tm_description/meshes/tm900/visual/Arm2.STL" />
+	  <mesh filename="package://tm_description/meshes/tm900/visual/Arm2.dae" />
         </geometry>
         <material name="DarkOlive">
@@ -167,5 +167,5 @@
       <visual>
         <geometry>
-	  <mesh filename="package://tm_description/meshes/tm900/visual/Wrist1.STL" />
+	  <mesh filename="package://tm_description/meshes/tm900/visual/Wrist1.dae" />
         </geometry>
         <material name="DarkOlive">
@@ -198,5 +198,5 @@
       <visual>
         <geometry>
-	  <mesh filename="package://tm_description/meshes/tm900/visual/Wrist2.STL" />
+	  <mesh filename="package://tm_description/meshes/tm900/visual/Wrist2.dae" />
         </geometry>
         <material name="DarkOlive">
@@ -229,5 +229,5 @@
       <visual>
         <geometry>
-	  <mesh filename="package://tm_description/meshes/tm900/visual/Wrist3.STL" />
+	  <mesh filename="package://tm_description/meshes/tm900/visual/Wrist3.dae" />
         </geometry>
 	<origin xyz="0 0 0.015" rpy="0 0 0"/>
